Commit message: done

File: src/sjtu_drone_description/urdf/sjtu_drone.urdf.xacro (robot description, xacro)
@@ -107,5 +107,5 @@
     <parent link="base_link"/>
     <child  link="red_cube_link"/>
-    <origin xyz="0 0 -0.15" rpy="0 0 0"/>
+    <origin xyz="0 0 -0.05" rpy="0 0 0"/>
   </joint>
   <!-- Ignition material (makes it red in Gazebo, not just RViz) -->
